File: MODULE-POWE-KAP2112K-V33D-01/MODULE-POWE-KAP2112K-V33D-01.kicad_sch (KiCad schematic)
At the start: 4 parts, among them U1 AP2112K-3.3

Commit message: Module massaging for IBBC-01
Other:
- note added: "MODULE-POWE KAP2112K-V33D-01 oom.lt/MPAP2112K"
Changed lines of the file:
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@@
     (stroke (width 0) (type default) (color 0 0 0 0))
+  )
+  (text "MODULE-POWE\nKAP2112K-V33D-01\noom.lt/MPAP2112K" (at 127 80.01 0)
+    (effects (font (size 3 3)) (justify left bottom))
   )
   (global_label "Vin" (shape input) (at 130.81 92.71 180) (fields_autoplaced)
