File: MODULE-CONN-BRBO-IBBC-SZ01/MODULE-CONN-BRBO-IBBC-SZ01.kicad_pcb (KiCad board)
At the start: 2 copper layers, 30 x 20 mm, 6 parts, among them J1 HEAD-I01-X-PI10-01 oom.lt/H10, J2 HEAD-I01-X-PI04-01 oom.lt/H4, J3 HEAD-JSTSH-X-PI04-RS oom.lt/H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, J4 HEAD-JSTSH-X-PI04-RS oom.lt/H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

Commit message: Worked on footprintification.
Parts:
- added U10: MODULE-CONN-BRBO-IBBC-SZ01, oomlout_OOMP_modules:MODULE-CONN-BRBO-IBBC-SZ01, F.Cu at (155.0, 137.5)
Routing:
- net SDA: track 0.00 -> 75.3 mm, vias 0 -> 4
- net SCL: track 0.00 -> 72.9 mm, vias 0 -> 4
- net +3V3: track 0.00 -> 30.7 mm, vias 0 -> 2
- net unconnected-(U10-Pad5): track 0.00 -> 30.7 mm, vias 0 -> 2
