File: MODULE-CONN-BRBO-IBBC-SZ01/MODULE-CONN-BRBO-IBBC-SZ01.kicad_sch (KiCad schematic)
At the start: 6 parts, among them J1 HEAD-I01-X-PI10-01 oom.lt/H10, J2 HEAD-I01-X-PI04-01 oom.lt/H4, J3 HEAD-JSTSH-X-PI04-RS oom.lt/H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, J4 HEAD-JSTSH-X-PI04-RS oom.lt/H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

Commit message: Worked on footprintification.
Parts:
- added U10: MODULE-CONN-BRBO-IBBC-SZ01, oomlout_OOMP_modules:MODULE-CONN-BRBO-IBBC-SZ01, symbol oomlout_OOMP_modules:MODULE-CONN-BRBO-IBBC-SZ01
Connections:
- net +3V3: now also U10.5 (3V3)
- net CS: now also U10.8 (CS)
- net EX01: now also U10.1 (EX01)
- net EX02: now also U10.2 (EX02)
- net EX03: now also U10.9 (EX03)
- net EX04: now also U10.10 (EX04)
- net EX05: now also U10.11 (EX05)
- net EX06: now also U10.12 (EX06)
- net EX07: now also U10.13 (EX07)
- net EX08: now also U10.14 (EX08)
- net GND: now also U10.4 (GND)
- net SCL: now also U10.7 (SCL)
- net SDA: now also U10.6 (SDA)
- net VCC: now also U10.3 (VCC)
Other:
- note added: "SIMPLIFIED"
- note added: "VERBOSE"
- moved on the sheet: H1, H2, J1, J2, J3, J4
